File: _autosave-DCDC5V20A.kicad_sch (KiCad schematic)
At the start: 35 parts, among them J1 Conn_01x02_Socket, J2 Conn_01x02_Socket, Q1 NMOS, Q2 NMOS

Commit message: edit layout
Parts:
- C12: value 4u7 -> 1u
Changed lines of the file:
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@@
       (effects (font (size 1.27 1.27)) (justify left))
     )
-    (property "Value" "4u7" (at 243.84 81.915 0)
+    (property "Value" "1u" (at 243.84 81.915 0)
       (effects (font (size 1.27 1.27)) (justify left))
     )
